File: Electricals/KCORES-FlexibleLOM-Adapter/KCORES-FlexibleLOM-Adapter.kicad_pcb (KiCad board)
At the start: 2 copper layers, 96.3 x 25.7 mm, 6 parts, among them J1 PCIe_x8, J2 HPE_FlexibleLOM

Commit message: v1.1
Connections:
- J1 pad B48: Net-(J1-PadB48) -> GND
- J2 pad A10: /SDP1_3 -> +3V3
- J2 pad A11: /SDP0_3 -> +3V3
Routing:
- net +3V3: track 53.7 -> 71.3 mm
- net +12V: track 69.3 -> 73.4 mm
- net GND: track 240.7 -> 243.4 mm, vias 131 -> 138
- net /nWAKE: track 35.9 -> 36.8 mm
Other:
- board text added: "V1.1"
- board text removed: "V1.0"
