File: Electricals/KCORES-FlexibleLOM-Adapter/KCORES-FlexibleLOM-Adapter.sch (KiCad schematic (older format))
At the start: 5 parts, among them J1 PCIe_x8, J2 HPE_FlexibleLOM

Commit message: v1.1
Connections:
- net SDP0_3 is gone; now on net +3V3: J2.A11 (Pin_A11)
- net SDP1_3 is gone; now on net +3V3: J2.A10 (Pin_A10)
- net GND: now also J1.B48 (Pin_B48)
- no-connect marks 30 -> 27
Changed lines of the file:
@@
 	2500 1600 2500 1500
 Connection ~ 2500 1500
-NoConn ~ 2250 1400
 NoConn ~ 1750 1800
 NoConn ~ 1750 1900
@@
 Text Label 2250 2600 0    50   ~ 0
 GND
-NoConn ~ 1750 6200
 NoConn ~ 1750 4500
 NoConn ~ 1750 3100
@@
 Wire Wire Line
 	7000 1800 7000 1900
-NoConn ~ 6250 2300
-NoConn ~ 6250 2400
 Wire Wire Line
 	6250 1400 7000 1400
@@
 NoConn ~ 9500 1650
 NoConn ~ 9500 2150
+$Comp
+L power:+3V3 #PWR0110
+U 1 1 5FAFCD0D
+P 6650 2300
+F 0 "#PWR0110" H 6650 2150 50  0001 C CNN
+F 1 "+3V3" H 6665 2473 50  0000 C CNN
+F 2 "" H 6650 2300 50  0001 C CNN
+F 3 "" H 6650 2300 50  0001 C CNN
+	1    6650 2300
+	-1   0    0    -1
+$EndComp
+Wire Wire Line
+	6650 2300 6250 2300
+Wire Wire Line
+	6250 2400 6650 2400
+Wire Wire Line
+	6650 2400 6650 2300
+Connection ~ 6650 2300
+Text Label 1750 6200 2    50   ~ 0
+GND
+NoConn ~ 2250 1400
 $EndSCHEMATC
